File: karabas_128_cpld.kicad_sch (KiCad schematic)
At the start: 11 parts, among them IC10 EPM7128STC100-15N, X6 JTAG

Commit message: small improvements
Parts:
- IC10: value EPM7128STC100-15N -> EPM7128STC100
Changed lines of the file:
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@@
       (effects (font (size 2.0828 1.7703)) (justify left bottom))
     )
-    (property "Value" "EPM7128STC100-15N" (at 117.8052 95.6056 0)
+    (property "Value" "EPM7128STC100" (at 117.8052 95.6056 0)
       (effects (font (size 2.0828 1.7703)) (justify left bottom))
     )

Commit message: WIP
Parts:
- U11: renamed from IC10; footprint karabas_128:QFP50P1600X1600X120-100N -> Package_QFP:TQFP-100_14x14mm_P0.5mm
Changed lines of the file:
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@@
     (stroke (width 0) (type default))
   )
-  (text "CPLD" (at 259.08 25.4 0)
-    (effects (font (size 5.08 4.318)) (justify left bottom))
+  (text "CPLD" (at 265.43 175.26 0)
+    (effects (font (size 3 3)) (justify left bottom))
   )
   (global_label "MD0" (shape bidirectional) (at 161.29 172.72 0) (fields_autoplaced)
@@
   (symbol (lib_id "karabas_128-eagle-import:EPM7128STC100-15N") (at 128.27 101.6 0) (unit 1)
     (in_bom yes) (on_board yes) (dnp no)
-    (property "Reference" "IC10" (at 122.7582 100.0506 0)
+    (property "Reference" "U11" (at 122.7582 100.0506 0)
       (effects (font (size 2.0828 1.7703)) (justify left bottom))
     )
@@
       (effects (font (size 2.0828 1.7703)) (justify left bottom))
     )
-    (property "Footprint" "karabas_128:QFP50P1600X1600X120-100N" (at 128.27 101.6 0)
+    (property "Footprint" "Package_QFP:TQFP-100_14x14mm_P0.5mm" (at 128.27 101.6 0)
       (effects (font (size 1.27 1.27)) hide)
     )
@@
       (project "karabas_128"
         (path "/70a04a89-960f-41bf-b5c3-0fa551716ed9/f627de00-92d5-4d33-b09b-85f1ce1ea363"
-          (reference "IC10") (unit 1)
-        )
-      )
+          (reference "U11") (unit 1)
+        )
+      )
